Commit message: client ik update

File: urdf/nova5_robot_panther_camera.xacro (robot description, xacro)
@@ -728,4 +728,11 @@
     <child link="base_link_gripper"/>
     <origin xyz="0.0 0.0 0.0" rpy="0 0 0"/>
+  </joint>
+  <!-- create a virtual fixed joint for having the point of the picking of the gripper-->
+ <link name="picking_point" />
+ <joint name="picking_joint" type="fixed">
+    <parent link="Link6"/>
+    <child link="picking_point"/>
+    <origin xyz="0.0 0.0 0.12" rpy="0 0 0"/>
   </joint>
  <xacro:macro name="robot_transmission" params="joint_name">
